Commit message: modeled EZArm in urdf,

File: src/testbot_description/urdf/my_robot.urdf (robot description, URDF)
Before this commit: robot test_robot, 4 links, 3 joints
Links:
- removed link link1
- removed link link2
- removed link link3
- removed link link4
- added link base_link; visual mesh filename=package://testbot_description/meshes/base_link.stl scale=.001 .001 .001
- added link claw_support; visual mesh filename=package://testbot_description/meshes/claw_support.stl scale=.001 .001 .001
- added link forearm_link; visual mesh filename=package://testbot_description/meshes/link.stl scale=.001 .001 .001
- added link forward_drive_arm; visual mesh filename=package://testbot_description/meshes/forward_drive_arm.stl scale=.001 .001 .001
- added link horizontal_arm; visual mesh filename=package://testbot_description/meshes/horizontal_arm.stl scale=.001 .001 .001
- added link main_mount; visual mesh filename=package://testbot_description/meshes/main_mount.stl scale=.001 .001 .001
- added link round_plate; visual mesh filename=package://testbot_description/meshes/round_plate.stl scale=.001 .001 .001
- added link static_link_1; visual mesh filename=package://testbot_description/meshes/link.stl scale=.001 .001 .001
- added link triangle_link; visual mesh filename=package://testbot_description/meshes/triangular_link.stl scale=.001 .001 .001
- added link vertical_drive_arm; visual mesh filename=package://testbot_description/meshes/vertical_drive_arm.stl scale=.001 .001 .001
- added link vertical_drive_link; visual mesh filename=package://testbot_description/meshes/link.stl scale=.001 .001 .001
- added link virtual_fwdDrive_horizArm; visual cylinder length=.01 radius=0.001
- added link virtual_vertDrive_link; visual cylinder length=.01 radius=0.001
Joints:
- removed joint joint1
- removed joint joint2
- removed joint joint3
- added joint claw_joint: type continuous, parent horizontal_arm, child claw_support, origin xyz=0 0.800 0 rpy=0 0 0, axis 1 0 0, mimic joint=vertical_servo multiplier=-1 offset=0
- added joint forearm_link_joint_a: type continuous, parent triangle_link, child forearm_link, origin xyz=-0.040 0.1723 -0.101553 rpy=-1.5708 0 0, axis 1 0 0, mimic joint=vertical_servo multiplier=1 offset=0
- added joint forward_servo: type continuous, parent main_mount, child forward_drive_arm, origin xyz=0.210 0 .304 rpy=0 0 0, axis 1 0 0
- added joint fwdArm_trianlge_joint: type continuous, parent forward_drive_arm, child triangle_link, origin xyz=0.088 0 0.800 rpy=1.5708 0 0, axis 1 0 0, mimic joint=forward_servo multiplier=-1 offset=0
- added joint fwd_drv_horiz_arm_a: type continuous, parent forward_drive_arm, child virtual_fwdDrive_horizArm, origin xyz=-0.092 0 0.800, axis 1 0 0, mimic joint=forward_servo multiplier=-1 offset=0
- added joint fwd_drv_horiz_arm_b: type continuous, parent virtual_fwdDrive_horizArm, child horizontal_arm, origin xyz=0 0 0, axis 1 0 0, mimic joint=vertical_servo multiplier=1 offset=0
- added joint plate_mount: type fixed, parent round_plate, child main_mount, origin xyz=-0.140 0 0.045 rpy=0 0 0
- added joint static_link_joint: type continuous, parent main_mount, child static_link_1, origin xyz=0.300 -0.361 0.4763 rpy=1.5708 0 0, axis 1 0 0, mimic joint=forward_servo multiplier=1 offset=0
- added joint vertDrive_link_a: type continuous, parent vertical_drive_arm, child virtual_vertDrive_link, origin xyz=0 0 .350, axis 1 0 0, mimic joint=forward_servo multiplier=1 offset=0
- added joint vertDrive_link_b: type continuous, parent virtual_vertDrive_link, child vertical_drive_link, origin xyz=0 0 0, axis 1 0 0, mimic joint=vertical_servo multiplier=-1 offset=0
- added joint vertical_servo: type continuous, parent main_mount, child vertical_drive_arm, origin xyz=.048 0 .304 rpy=1.5708 0 0, axis 1 0 0
- added joint yaw_servo: type continuous, parent base_link, child round_plate, origin xyz=0 0 .310, axis 0 0 1
